File: KiCad/projects/concentrador2/PCB_Project.kicad_pcb (KiCad board)
At the start: 2 copper layers, 91.4 x 88 mm, 43 parts, among them J1 54602-908LF, P1 Grabador, P2 Entrada fuente externa, P4 Header 20X2, P5 Header 2, U1 DSPIC33EP256MC202-I/SP, U2 STEP_DOWN_CONVERTER, U3 LD33V, U4 MAX485, U5 DS3234S#, U9 MAX485

Commit message: PCB Acelerografo & Nodo
Parts:
- added REF**: Fiducial_1mm_Mask2mm, Fiducial:Fiducial_1mm_Mask2mm, F.Cu at (184.7, 69.0)
- added REF**: Fiducial_1mm_Mask2mm, Fiducial:Fiducial_1mm_Mask2mm, F.Cu at (172.8, 147.0)
- added REF**: Fiducial_1mm_Mask2mm, Fiducial:Fiducial_1mm_Mask2mm, F.Cu at (106.5, 143.9)
- added REF**: Fiducial_1mm_Mask2mm, Fiducial:Fiducial_1mm_Mask2mm, F.Cu at (108.0, 74.3)
- U5: moved to F.Cu
Routing:
- net NetBT1_0: track 85.0 -> 51.5 mm, vias 1 -> 2
- net VCC: track 239.7 -> 271.0 mm, vias 4 -> 6
- net GND: track 517.5 -> 501.0 mm, vias 1 -> 2
- net SINC_A: track 49.3 -> 32.9 mm
- net SPI2_MOSI: track 14.7 -> 30.3 mm
- net 5V: track 177.9 -> 162.8 mm, vias 2 -> 4
- net SINC_B: track 53.8 -> 39.5 mm
- net RPI_INT1: track 106.4 -> 118.7 mm
- net SPI2_DS3234_CS: track 24.4 -> 36.4 mm, vias 1 -> 3
- net SPI2_MISO: track 33.3 -> 45.0 mm, vias 0 -> 1
- net DS3231_SQW: track 60.6 -> 50.9 mm, vias 1 -> 0
- net DSPIC_TX: track 70.1 -> 79.5 mm
- net A: track 46.8 -> 56.1 mm, vias 2 -> 1
- net GPS_1PPS: track 60.5 -> 69.2 mm, vias 1 -> 2
- net FUENTE_12V: track 85.8 -> 78.7 mm
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Other:
- board text added: "Acelerografo V2.2.0"
- board text removed: "Acelerografo V1.4"
- board text removed: "v24.2.27"

Commit message: Cambios Finales en PCB's
Parts:
- removed D1: 1N914, Diode_THT:D_DO-35_SOD27_P7.62mm_Horizontal
- removed the REF** at (184.7, 69.0)
- removed the REF** at (172.8, 147.0)
- removed the REF** at (106.5, 143.9)
- removed the REF** at (108.0, 74.3)
- added D3: 1N4148WS, Diode_SMD:D_SOD-323, F.Cu at (116.9, 119.0)
- added REF**: Fiducial_1mm_Mask2mm, Fiducial:Fiducial_1mm_Mask2mm, F.Cu at (184.2, 68.7)
- added REF**: Fiducial_1mm_Mask2mm, Fiducial:Fiducial_1mm_Mask2mm, F.Cu at (106.5, 74.3)
- added REF**: Fiducial_1mm_Mask2mm, Fiducial:Fiducial_1mm_Mask2mm, F.Cu at (143.0, 145.7)
- BT2: footprint Battery:BatteryHolder_Keystone_500 -> CR1220:CR1220-2
- moved BT2 5.48 mm to (145.8, 95.1), turned to 180 degrees
Routing:
- net DS3231_SQW: track 50.9 -> 81.6 mm, vias 0 -> 2
- net RPI_INT1: track 118.7 -> 102.7 mm, vias 0 -> 1
- net GND: track 501.0 -> 513.4 mm, vias 2 -> 4
- net A: track 56.1 -> 44.5 mm, vias 1 -> 2
- net SPI2_DS3234_CS: track 36.4 -> 46.0 mm
- net DSPIC_TX: track 79.5 -> 70.7 mm, vias 0 -> 1
- net NetBT1_0: track 51.5 -> 43.5 mm
- net VCC: track 271.0 -> 264.1 mm, vias 6 -> 3
- net B: track 46.7 -> 40.0 mm
- net SPI1_MISO: track 92.5 -> 87.5 mm, vias 0 -> 2
- net INT_SINC_1: track 32.9 -> 37.8 mm
- net 5V: track 162.8 -> 166.8 mm, vias 4 -> 2
- net _DSPIC_RX: track 66.5 -> 63.2 mm
- net GPS_1PPS: track 69.2 -> 66.2 mm
- net SPI2_MOSI: track 30.3 -> 32.9 mm, vias 0 -> 3
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
Commit message: Cambios en el PCB
Parts:
- removed REF** (x3): Fiducial_1mm_Mask2mm, Fiducial:Fiducial_1mm_Mask2mm
- BT2: footprint CR1220:CR1220-2 -> LibExt:CR1220-2-ext
- C10: value Cap -> 1uF
- C12, C13, C15: value Cap -> 100nF
- R1, R16, R18: value Res1 -> 1K
- R14, R2, R5: value Res1 -> 3K3
- R17: value Res1 -> 10K
- R3: value Res1 -> 4K7
- R4: value Res1 -> 100K
