File: KiCad/projects/concentrador2/PCB_Project.kicad_sch (KiCad schematic)
At the start: 43 parts, among them J1 54602-908LF, P1 Grabador, P2 Entrada fuente externa, P4 Header 20X2, P5 Header 2, U1 DSPIC33EP256MC202-I/SP, U2 STEP_DOWN_CONVERTER, U3 LD33V, U4 MAX485, U5 DS3234S#, U9 MAX485

Commit message: Cambios Finales en PCB's
Parts:
- removed D1: 1N914, Diode_THT:D_DO-35_SOD27_P7.62mm_Horizontal, symbol Diode:1N914
- added D3: 1N4148WS, Diode_SMD:D_SOD-323, symbol Diode:1N4148WS
- BT2: footprint Battery:BatteryHolder_Keystone_500 -> CR1220:CR1220-2; LCSC (none) -> C70381; now in the parts list
Connections:
- net VCC: now also D3.2 (A)
- net at R3.2: now also D3.1 (K)
Changed lines of the file:
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@@
 	(wire
 		(pts
+			(xy 35.56 116.6622) (xy 35.56 118.11)
+		)
+		(stroke
+			(width 0)
+			(type default)
+		)
+	)
+	(wire
+		(pts
 			(xy 317.5 214.63) (xy 312.42 214.63)
 		)
@@
 	(wire
 		(pts
+			(xy 49.784 118.11) (xy 55.88 118.11)
+		)
+		(stroke
+			(width 0)
+			(type default)
+		)
+	)
+	(wire
+		(pts
 			(xy 93.98 196.85) (xy 99.06 196.85)
 		)
@@
 	(wire
 		(pts
-			(xy 49.53 118.11) (xy 55.88 118.11)
-		)
-		(stroke
-			(width 0)
-			(type default)
-		)
-	)
-	(wire
-		(pts
 			(xy 360.68 80.264) (xy 360.68 81.026)
 		)
@@
 	(wire
 		(pts
-			(xy 35.56 116.6622) (xy 35.56 118.11)
-		)
-		(stroke
-			(width 0)
-			(type default)
-		)
-	)
-	(wire
-		(pts
 			(xy 99.06 195.4022) (xy 99.06 196.85)
 		)
@@
 	(wire
 		(pts
+			(xy 35.56 118.11) (xy 42.164 118.11)
+		)
+		(stroke
+			(width 0)
+			(type default)
+		)
+	)
+	(wire
+		(pts
 			(xy 132.08 83.6422) (xy 129.54 83.6422)
 		)
@@
 	(wire
 		(pts
-			(xy 41.91 118.11) (xy 35.56 118.11)
-		)
-		(stroke
-			(width 0)
-			(type default)
-		)
-	)
-	(wire
-		(pts
 			(xy 360.68 73.4822) (xy 358.14 73.4822)
 		)
@@
 	)
 	(symbol
+		(lib_id "Diode:1N4148WS")
+		(at 45.974 118.11 180)
+		(unit 1)
+		(body_style 1)
+		(exclude_from_sim no)
+		(in_bom yes)
+		(on_board yes)
+		(in_pos_files yes)
+		(dnp no)
+		(property "Reference" "D3"
+			(at 45.974 111.76 0)
+			(show_name no)
+			(do_not_autoplace no)
+			(effects
+				(font
+					(size 1.27 1.27)
+				)
+			)
+		)
+		(property "Value" "1N4148WS"
+			(at 45.974 114.3 0)
+			(show_name no)
+			(do_not_autoplace no)
+			(effects
+				(font
+					(size 1.27 1.27)
+				)
+			)
+		)
+		(property "Footprint" "Diode_SMD:D_SOD-323"
+			(at 45.974 113.665 0)
+			(hide yes)
+			(show_name no)
+			(do_not_autoplace no)
+			(effects
+				(font
+					(size 1.27 1.27)
+				)
+			)
+		)
+		(property "Datasheet" "https://www.vishay.com/docs/85751/1n4148ws.pdf"
+			(at 45.974 118.11 0)
+			(hide yes)
+			(show_name no)
+			(do_not_autoplace no)
+			(effects
+				(font
+					(size 1.27 1.27)
+				)
+			)
+		)
+		(property "Description" "75V 0.15A Fast switching Diode, SOD-323"
+			(at 45.974 118.11 0)
+			(hide yes)
+			(show_name no)
+			(do_not_autoplace no)
+			(effects
+				(font
+					(size 1.27 1.27)
+				)
+			)
+		)
+		(property "Sim.Device" "D"
+			(at 45.974 118.11 0)
+			(hide yes)
+			(show_name no)
+			(do_not_autoplace no)
+			(effects
+				(font
+					(size 1.27 1.27)
+				)
+			)
+		)
+		(property "Sim.Pins" "1=K 2=A"
+			(at 45.974 118.11 0)
+			(hide yes)
+			(show_name no)
+			(do_not_autoplace no)
+			(effects
+				(font
+					(size 1.27 1.27)
+				)
+			)
+		)
+		(property "LCSC" "C2128"
+			(at 45.974 116.078 0)
+			(show_name no)
+			(do_not_autoplace no)
+			(effects
+				(font
+					(size 1.27 1.27)
+				)
+			)
+		)
+		(pin "1"
+		)
+		(pin "2"
+		)
+		(instances
+			(project "PCB_Project"
+				(path "/0dc9dba4-ff0b-442b-8d95-98389b6a93ed"
+					(reference "D3")
+					(unit 1)
+				)
+			)
+		)
+	)
+	(symbol
 		(lib_id "PCB_Project-altium-import:GND_POWER_GROUND")
 		(at 342.9 50.6222 0)
@@
 		(body_style 1)
 		(exclude_from_sim no)
-		(in_bom no)
+		(in_bom yes)
 		(on_board yes)
-		(in_pos_files no)
+		(in_pos_files yes)
 		(dnp no)
-		(fields_autoplaced yes)
 		(property "Reference" "BT2"
 			(at 393.446 86.0424 0)
@@
 			)
 		)
-		(property "Footprint" "Battery:BatteryHolder_Keystone_500"
+		(property "Footprint" "CR1220:CR1220-2"
 			(at 389.636 86.36 90)
 			(hide yes)
@@
 			)
 		)
+		(property "LCSC" "C70381"
+			(at 397.002 90.932 0)
+			(show_name no)
+			(do_not_autoplace no)
+			(effects
+				(font
+					(size 1.27 1.27)
+				)
+			)
+		)
 		(pin "2"
 		)
@@
 					(unit 1)
 				)
-			)
-		)
-	)
-	(symbol
-		(lib_id "Diode:1N914")
-		(at 45.72 118.11 180)
-		(unit 1)
-		(body_style 1)
-		(exclude_from_sim no)
-		(in_bom no)
-		(on_board yes)
-		(in_pos_files no)
-		(dnp no)
-		(fields_autoplaced yes)
-		(property "Reference" "D1"
-			(at 45.72 111.76 0)
-			(show_name no)
-			(do_not_autoplace no)
-			(effects
-				(font
-					(size 1.27 1.27)
-				)
-			)
-		)
-		(property "Value" "1N914"
-			(at 45.72 114.3 0)
-			(show_name no)
-			(do_not_autoplace no)
-			(effects
-				(font
-					(size 1.27 1.27)
-				)
-			)
-		)
-		(property "Footprint" "Diode_THT:D_DO-35_SOD27_P7.62mm_Horizontal"
-			(at 45.72 113.665 0)
-			(hide yes)
-			(show_name no)
-			(do_not_autoplace no)
-			(effects
-				(font
-					(size 1.27 1.27)
-				)
-			)
-		)
-		(property "Datasheet" "http://www.vishay.com/docs/85622/1n914.pdf"
-			(at 45.72 118.11 0)
-			(hide yes)
-			(show_name no)
-			(do_not_autoplace no)
-			(effects
-				(font
-					(size 1.27 1.27)
-				)
-			)
-		)
-		(property "Description" "100V 0.3A Small Signal Fast Switching Diode, DO-35"
-			(at 45.72 118.11 0)
-			(hide yes)
-			(show_name no)
-			(do_not_autoplace no)
-			(effects
-				(font
-					(size 1.27 1.27)
-				)
-			)
-		)
-		(property "Sim.Device" "D"
-			(at 45.72 118.11 0)
-			(hide yes)
-			(show_name no)
-			(do_not_autoplace no)
-			(effects
-				(font
-					(size 1.27 1.27)
-				)
-			)
-		)
-		(property "Sim.Pins" "1=K 2=A"
-			(at 45.72 118.11 0)
-			(hide yes)
-			(show_name no)
-			(do_not_autoplace no)
-			(effects
-				(font
-					(size 1.27 1.27)
-				)
-			)
-		)
-		(pin "2"
-		)
-		(pin "1"
-		)
-		(instances
-			(project "PCB_Project"
-				(path "/0dc9dba4-ff0b-442b-8d95-98389b6a93ed"
-					(reference "D1")
-					(unit 1)
-				)

Commit message: Cambios en el PCB
Parts:
- C1: ALTIUM_VALUE 470uF -> (none); LATESTREVISIONDATE 17-Jul-2002 -> (none); LATESTREVISIONNOTE Re-released for DXP Platform. -> (none); PACKAGEDESCRIPTION Radial Cap, Thru-Hole; 2 Leads; 0.3 in Pin Spacing -> (none); PACKAGEREFERENCE RAD-0.3 -> (none); PUBLISHED 8-Jun-2000 -> (none); PUBLISHER Altium Limited -> (none)
- C10: value Cap -> 1uF; ALTIUM_VALUE 1uF -> (none); LATESTREVISIONDATE 17-Jul-2002 -> (none); LATESTREVISIONNOTE Re-released for DXP Platform. -> (none); PACKAGEDESCRIPTION Radial Cap, Thru-Hole; 2 Leads; 0.3 in Pin Spacing -> (none); PACKAGEREFERENCE RAD-0.3 -> (none); PUBLISHED 8-Jun-2000 -> (none); PUBLISHER Altium Limited -> (none)
- C12, C13, C15: value Cap -> 100nF; ALTIUM_VALUE 100nF -> (none); LATESTREVISIONDATE 17-Jul-2002 -> (none); LATESTREVISIONNOTE Re-released for DXP Platform. -> (none); PACKAGEDESCRIPTION Radial Cap, Thru-Hole; 2 Leads; 0.3 in Pin Spacing -> (none); PACKAGEREFERENCE RAD-0.3 -> (none); PUBLISHED 8-Jun-2000 -> (none); PUBLISHER Altium Limited -> (none)
- C2, C4, C5, C7, C8: ALTIUM_VALUE 100nF -> (none); LATESTREVISIONDATE 17-Jul-2002 -> (none); LATESTREVISIONNOTE Re-released for DXP Platform. -> (none); PACKAGEDESCRIPTION Radial Cap, Thru-Hole; 2 Leads; 0.3 in Pin Spacing -> (none); PACKAGEREFERENCE RAD-0.3 -> (none); PUBLISHED 8-Jun-2000 -> (none); PUBLISHER Altium Limited -> (none)
- C3: ALTIUM_VALUE 220uF -> (none); LATESTREVISIONDATE 17-Jul-2002 -> (none); LATESTREVISIONNOTE Re-released for DXP Platform. -> (none); PACKAGEDESCRIPTION Radial Cap, Thru-Hole; 2 Leads; 0.3 in Pin Spacing -> (none); PACKAGEREFERENCE RAD-0.3 -> (none); PUBLISHED 8-Jun-2000 -> (none); PUBLISHER Altium Limited -> (none)
- C6, C9: ALTIUM_VALUE 10nF -> (none); LATESTREVISIONDATE 17-Jul-2002 -> (none); LATESTREVISIONNOTE Re-released for DXP Platform. -> (none); PACKAGEDESCRIPTION Radial Cap, Thru-Hole; 2 Leads; 0.3 in Pin Spacing -> (none); PACKAGEREFERENCE RAD-0.3 -> (none); PUBLISHED 8-Jun-2000 -> (none); PUBLISHER Altium Limited -> (none)
- D2, D4, D5: DATASHEETVERSION 16-Apr-2002 -> (none); LATESTREVISIONDATE 17-Dec-2003 -> (none); LATESTREVISIONNOTE PCB Footprint replaced. -> (none); PACKAGEDESCRIPTION SM LED; 2 C-Bend Leads; Body 3.5 x 2.8 x 1.9 mm, inc leads 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 -> (none); PACKAGEREFERENCE 3.5X2.8X1.9 -> (none); PACKAGEVERSION 16-Apr-2002 -> (none); PUBLISHED 8-Jun-2000 -> (none); PUBLISHER Altium Limited -> (none)
- J1: ALTIUM_VALUE * -> (none); DIGI-KEY_PART_NUMBER 609-1046-ND -> (none); DIGI-KEY_PURCHASE_URL https://www.digikey.com/product-detail/en/amphenol-icc-fci/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 -> (none); MF Amphenol ICC -> (none); MP 54602-908LF -> (none); SNAPEDA_LINK https://www.snapeda.com/parts/54602-908LF/Amphenol%20FCI/vi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 -> (none)
- P1, P2, P4, P5: LATESTREVISIONDATE 17-Jul-2002 -> (none); LATESTREVISIONNOTE Re-released for DXP Platform. -> (none); PUBLISHER Altium Limited -> (none)
- R1, R16, R18: value Res1 -> 1K; ALTIUM_VALUE 1K -> (none); LATESTREVISIONDATE 17-Jul-2002 -> (none); LATESTREVISIONNOTE Re-released for DXP Platform. -> (none); PACKAGEDESCRIPTION Axial Device, Thru-Hole; 2 Leads; 0.3 in Pin Spacing -> (none); PACKAGEREFERENCE AXIAL-0.3 -> (none); PUBLISHED 8-Jun-2000 -> (none); PUBLISHER Altium Limited -> (none)
- R13: ALTIUM_VALUE 3K3 -> (none); LATESTREVISIONDATE 17-Jul-2002 -> (none); LATESTREVISIONNOTE Re-released for DXP Platform. -> (none); PACKAGEDESCRIPTION Axial Device, Thru-Hole; 2 Leads; 0.3 in Pin Spacing -> (none); PACKAGEREFERENCE AXIAL-0.3 -> (none); PUBLISHED 8-Jun-2000 -> (none); PUBLISHER Altium Limited -> (none)
- R14, R2, R5: value Res1 -> 3K3; ALTIUM_VALUE 3K3 -> (none); LATESTREVISIONDATE 17-Jul-2002 -> (none); LATESTREVISIONNOTE Re-released for DXP Platform. -> (none); PACKAGEDESCRIPTION Axial Device, Thru-Hole; 2 Leads; 0.3 in Pin Spacing -> (none); PACKAGEREFERENCE AXIAL-0.3 -> (none); PUBLISHED 8-Jun-2000 -> (none); PUBLISHER Altium Limited -> (none)
- R15: ALTIUM_VALUE 10K -> (none); LATESTREVISIONDATE 17-Jul-2002 -> (none); LATESTREVISIONNOTE Re-released for DXP Platform. -> (none); PACKAGEDESCRIPTION Axial Device, Thru-Hole; 2 Leads; 0.3 in Pin Spacing -> (none); PACKAGEREFERENCE AXIAL-0.3 -> (none); PUBLISHED 8-Jun-2000 -> (none); PUBLISHER Altium Limited -> (none)
- R17: value Res1 -> 10K; ALTIUM_VALUE 10K -> (none); LATESTREVISIONDATE 17-Jul-2002 -> (none); LATESTREVISIONNOTE Re-released for DXP Platform. -> (none); PACKAGEDESCRIPTION Axial Device, Thru-Hole; 2 Leads; 0.3 in Pin Spacing -> (none); PACKAGEREFERENCE AXIAL-0.3 -> (none); PUBLISHED 8-Jun-2000 -> (none); PUBLISHER Altium Limited -> (none)
- R3: value Res1 -> 4K7; ALTIUM_VALUE 4K7 -> (none); LATESTREVISIONDATE 17-Jul-2002 -> (none); LATESTREVISIONNOTE Re-released for DXP Platform. -> (none); PACKAGEDESCRIPTION Axial Device, Thru-Hole; 2 Leads; 0.3 in Pin Spacing -> (none); PACKAGEREFERENCE AXIAL-0.3 -> (none); PUBLISHED 8-Jun-2000 -> (none); PUBLISHER Altium Limited -> (none)
- R4: value Res1 -> 100K; ALTIUM_VALUE 100K -> (none); LATESTREVISIONDATE 17-Jul-2002 -> (none); LATESTREVISIONNOTE Re-released for DXP Platform. -> (none); PACKAGEDESCRIPTION Axial Device, Thru-Hole; 2 Leads; 0.3 in Pin Spacing -> (none); PACKAGEREFERENCE AXIAL-0.3 -> (none); PUBLISHED 8-Jun-2000 -> (none); PUBLISHER Altium Limited -> (none)
- S1: LATESTREVISIONDATE 17-Jul-2002 -> (none); LATESTREVISIONNOTE Re-released for DXP Platform. -> (none); PACKAGEDESCRIPTION Switch; 2 Leads -> (none); PACKAGEREFERENCE SPST-2 -> (none); PUBLISHED 24-Mar-1999 -> (none); PUBLISHER Altium Limited -> (none)
- U1: COMPONENTLINK1DESCRIPTION Manufacturer URL -> (none); COMPONENTLINK1URL http://www.microchip.com -> (none); COMPONENTLINK2DESCRIPTION Datasheet -> (none); COMPONENTLINK2URL http://ww1.microchip.com/downloads/en/DeviceDoc/70657F.pdf -> (none); COMPONENTLINK3DESCRIPTION Package Specification -> (none); COMPONENTLINK3URL http://www.microchip.com/stellent/groups/techpub_sg/documen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 -> (none); COMPONENTLINK4DESCRIPTION Product URL -> (none); COMPONENTLINK4URL http://www.microchip.com/dsPIC33EP256MC202 -> (none); DATASHEETVERSION Rev. F -> (none); MOUNTING TECHNOLOGY Through Hole -> (none); PACKAGEDESCRIPTION 28-Lead Plastic Dual In-Line, 34.86 x 6.79 mm Body, 2.54 mm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 -> (none); PACKAGEREFERENCE SPDIP-SP28 -> (none); PACKAGEVERSION C04-070B -> (none); PARTNUMBER DSPIC33EP256MC202-I/SP -> (none); SUPPLIER 1 Digi-Key -> (none); SUPPLIER 2 Farnell -> (none); SUPPLIER 3 Newark -> (none); SUPPLIER 4 Mouser -> (none); SUPPLIER PART NUMBER 1 DSPIC33EP256MC202-I/SP-ND -> (none); SUPPLIER PART NUMBER 2 2212194 -> (none); SUPPLIER PART NUMBER 3 66T8001 -> (none); SUPPLIER PART NUMBER 4 579-PC33256MC202ISP -> (none)
- U5: ALTIUM_VALUE Value -> (none); BUILT_BY EMA_UL_Team -> (none); COPYRIGHT Copyright (C) 2018 Accelerated Designs. All rights reserved -> (none); REFDES RefDes -> (none); TYPE DEV -> (none); VENDOR Maxim Integrated Products -> (none)
- W1: LATESTREVISIONDATE 17-Jul-2002 -> (none); LATESTREVISIONNOTE Re-released for DXP Platform. -> (none); PACKAGEDESCRIPTION Radial Cap, Thru-Hole; 2 Leads; 0.2 in Pin Spacing -> (none); PACKAGEREFERENCE RAD-0.2 -> (none); PUBLISHED 24-Mar-1999 -> (none); PUBLISHER Altium Limited -> (none)
