File: KiCad/projects/nodo/R-007 ACELEROGRAFO ADXL355 V5.kicad_pcb (KiCad board)
At the start: 2 copper layers, 84.9 x 66.1 mm, 33 parts, among them J1 ${ALTIUM_VALUE}${VALUEAUX}, J2 54602-908LF, J3 54602-908LF, P1 Grabador, U1 DSPIC33EP256MC202-I/SP, U2 LM1117DT-5.0NOPB, U3 LD33V, U4 ADXL355Z, U5 MAX485, U6 LM7805_TO220, U9 MAX485

Commit message: PCB Acelerografo & Nodo
Parts:
- added REF**: Fiducial_1mm_Mask2mm, Fiducial:Fiducial_1mm_Mask2mm, F.Cu at (146.7, 75.0)
- added REF**: Fiducial_1mm_Mask2mm, Fiducial:Fiducial_1mm_Mask2mm, F.Cu at (115.2, 84.7)
- added REF**: Fiducial_1mm_Mask2mm, Fiducial:Fiducial_1mm_Mask2mm, F.Cu at (187.3, 135.7)
- added REF**: Fiducial_1mm_Mask2mm, Fiducial:Fiducial_1mm_Mask2mm, F.Cu at (116.5, 135.7)
Routing:
- net TEST1: track 33.3 -> 8.85 mm
- net SPI2_MOSI: track 57.5 -> 72.4 mm, vias 0 -> 1
- net INT_SINC: track 43.0 -> 56.6 mm
- net 5V: track 106.0 -> 119.2 mm, vias 3 -> 2
- net A: track 55.3 -> 44.0 mm
- net DSPIC_RX: track 26.3 -> 35.7 mm
- net SPI1_SCK: track 23.8 -> 14.8 mm
- net SINC_B: track 45.9 -> 54.2 mm
- net VCC: track 161.2 -> 169.2 mm, vias 3 -> 2
- net SPI1_MOSI: track 23.7 -> 16.3 mm
- net SPI1_DSPIC_SS: track 46.7 -> 40.9 mm, vias 1 -> 0
- net FUENTE_12V: track 94.6 -> 90.1 mm
- net SINC_A: track 52.1 -> 56.5 mm, vias 0 -> 2
- net B: track 48.1 -> 44.9 mm
- net SPI2_MISO: track 33.7 -> 30.5 mm
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- added copper zone on B.Cu, net GND
- added copper zone on F.Cu, net GND
Other:
- board text added: "Acelerografo V2.2.0"
- board text removed: "Acelerografo V1.4"

Commit message: Cambios Finales en PCB's
Parts:
- removed the REF** at (146.7, 75.0)
- removed the REF** at (115.2, 84.7)
- removed the REF** at (187.3, 135.7)
- removed the REF** at (116.5, 135.7)
- added REF**: Fiducial_1mm_Mask2mm, Fiducial:Fiducial_1mm_Mask2mm, F.Cu at (117.2, 135.7)
- added REF**: Fiducial_1mm_Mask2mm, Fiducial:Fiducial_1mm_Mask2mm, F.Cu at (188.6, 136.5)
- added REF**: Fiducial_1mm_Mask2mm, Fiducial:Fiducial_1mm_Mask2mm, F.Cu at (147.7, 75.0)
- added REF**: Fiducial_1mm_Mask2mm, Fiducial:Fiducial_1mm_Mask2mm, F.Cu at (114.9, 84.9)
Routing:
- net VCC: track 169.2 -> 225.1 mm, vias 2 -> 4
- net A: track 44.0 -> 57.7 mm, vias 0 -> 3
- net SINC_A: track 56.5 -> 64.7 mm
- net SPI2_SCK: track 49.7 -> 57.0 mm
- net MCLR: track 74.5 -> 68.0 mm
- net 5V: track 119.2 -> 112.9 mm
- net GND: track 386.6 -> 380.5 mm, vias 5 -> 4
- net SINC_B: track 54.2 -> 48.8 mm, vias 0 -> 3
- net DSPIC_TX: track 28.0 -> 33.2 mm
- net _PGEC1: track 61.1 -> 66.2 mm, vias 0 -> 2
- net INT_SINC: track 56.6 -> 60.9 mm
- net DSPIC_RX: track 35.7 -> 31.6 mm
- net _PGED1: track 55.5 -> 59.5 mm
- net B: track 44.9 -> 41.0 mm
- net SPI2_MOSI: track 72.4 -> 69.8 mm
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