File: KiCad/projects/nodo/R-007 ACELEROGRAFO ADXL355 V5.kicad_sch (KiCad schematic)
At the start: 33 parts, among them J1 ${ALTIUM_VALUE}${VALUEAUX}, J2 54602-908LF, J3 54602-908LF, P1 Grabador, U1 DSPIC33EP256MC202-I/SP, U2 LM1117DT-5.0NOPB, U3 LD33V, U4 ADXL355Z, U5 MAX485, U6 LM7805_TO220, U9 MAX485

Commit message: Cambios en el PCB
Parts:
- C1: value Cap -> 470uF; ALTIUM_VALUE 470uF -> (none); LATESTREVISIONDATE 17-Jul-2002 -> (none); LATESTREVISIONNOTE Re-released for DXP Platform. -> (none); PACKAGEDESCRIPTION Radial Cap, Thru-Hole; 2 Leads; 0.3 in Pin Spacing -> (none); PACKAGEREFERENCE RAD-0.3 -> (none); PUBLISHED 8-Jun-2000 -> (none); PUBLISHER Altium Limited -> (none)
- C10: value Cap -> 1uF; ALTIUM_VALUE 1uF -> (none); LATESTREVISIONDATE 17-Jul-2002 -> (none); LATESTREVISIONNOTE Re-released for DXP Platform. -> (none); PACKAGEDESCRIPTION Radial Cap, Thru-Hole; 2 Leads; 0.3 in Pin Spacing -> (none); PACKAGEREFERENCE RAD-0.3 -> (none); PUBLISHED 8-Jun-2000 -> (none); PUBLISHER Altium Limited -> (none)
- C11, C13, C16, C2, C4, C5, C7, C8: value Cap -> 100nF; ALTIUM_VALUE 100nF -> (none); LATESTREVISIONDATE 17-Jul-2002 -> (none); LATESTREVISIONNOTE Re-released for DXP Platform. -> (none); PACKAGEDESCRIPTION Radial Cap, Thru-Hole; 2 Leads; 0.3 in Pin Spacing -> (none); PACKAGEREFERENCE RAD-0.3 -> (none); PUBLISHED 8-Jun-2000 -> (none); PUBLISHER Altium Limited -> (none)
- C3: value Cap -> 220uF; ALTIUM_VALUE 220uF -> (none); LATESTREVISIONDATE 17-Jul-2002 -> (none); LATESTREVISIONNOTE Re-released for DXP Platform. -> (none); PACKAGEDESCRIPTION Radial Cap, Thru-Hole; 2 Leads; 0.3 in Pin Spacing -> (none); PACKAGEREFERENCE RAD-0.3 -> (none); PUBLISHED 8-Jun-2000 -> (none); PUBLISHER Altium Limited -> (none)
- C6, C9: value Cap -> 10nF; ALTIUM_VALUE 10nF -> (none); LATESTREVISIONDATE 17-Jul-2002 -> (none); LATESTREVISIONNOTE Re-released for DXP Platform. -> (none); PACKAGEDESCRIPTION Radial Cap, Thru-Hole; 2 Leads; 0.3 in Pin Spacing -> (none); PACKAGEREFERENCE RAD-0.3 -> (none); PUBLISHED 8-Jun-2000 -> (none); PUBLISHER Altium Limited -> (none)
- D3: DATASHEETVERSION 16-Apr-2002 -> (none); LATESTREVISIONDATE 17-Dec-2003 -> (none); LATESTREVISIONNOTE PCB Footprint replaced. -> (none); PACKAGEDESCRIPTION SM LED; 2 C-Bend Leads; Body 3.5 x 2.8 x 1.9 mm, inc leads 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 -> (none); PACKAGEREFERENCE 3.5X2.8X1.9 -> (none); PACKAGEVERSION 16-Apr-2002 -> (none); PUBLISHED 8-Jun-2000 -> (none); PUBLISHER Altium Limited -> (none)
- J1: value ${ALTIUM_VALUE}${VALUEAUX} -> (none)
- J2, J3: ALTIUM_VALUE * -> (none); DIGI-KEY_PART_NUMBER 609-1046-ND -> (none); DIGI-KEY_PURCHASE_URL https://www.digikey.com/product-detail/en/amphenol-icc-fci/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 -> (none); MF Amphenol ICC -> (none); MP 54602-908LF -> (none); SNAPEDA_LINK https://www.snapeda.com/parts/54602-908LF/Amphenol%20FCI/vi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 -> (none); now left out of the parts list
- P1: LATESTREVISIONDATE 17-Jul-2002 -> (none); LATESTREVISIONNOTE Re-released for DXP Platform. -> (none); PUBLISHER Altium Limited -> (none); now left out of the parts list
- R1, R13, R14, R2: value Res1 -> 3K3; ALTIUM_VALUE 3K3 -> (none); LATESTREVISIONDATE 17-Jul-2002 -> (none); LATESTREVISIONNOTE Re-released for DXP Platform. -> (none); PACKAGEDESCRIPTION Axial Device, Thru-Hole; 2 Leads; 0.3 in Pin Spacing -> (none); PACKAGEREFERENCE AXIAL-0.3 -> (none); PUBLISHED 8-Jun-2000 -> (none); PUBLISHER Altium Limited -> (none)
- R3: value Res1 -> 4K7; ALTIUM_VALUE 4K7 -> (none); LATESTREVISIONDATE 17-Jul-2002 -> (none); LATESTREVISIONNOTE Re-released for DXP Platform. -> (none); PACKAGEDESCRIPTION Axial Device, Thru-Hole; 2 Leads; 0.3 in Pin Spacing -> (none); PACKAGEREFERENCE AXIAL-0.3 -> (none); PUBLISHED 8-Jun-2000 -> (none); PUBLISHER Altium Limited -> (none)
- R4: value Res1 -> 10K; ALTIUM_VALUE 10K -> (none); LATESTREVISIONDATE 17-Jul-2002 -> (none); LATESTREVISIONNOTE Re-released for DXP Platform. -> (none); PACKAGEDESCRIPTION Axial Device, Thru-Hole; 2 Leads; 0.3 in Pin Spacing -> (none); PACKAGEREFERENCE AXIAL-0.3 -> (none); PUBLISHED 8-Jun-2000 -> (none); PUBLISHER Altium Limited -> (none)
- R6: value Res1 -> 1K; ALTIUM_VALUE 1K -> (none); LATESTREVISIONDATE 17-Jul-2002 -> (none); LATESTREVISIONNOTE Re-released for DXP Platform. -> (none); PACKAGEDESCRIPTION Axial Device, Thru-Hole; 2 Leads; 0.3 in Pin Spacing -> (none); PACKAGEREFERENCE AXIAL-0.3 -> (none); PUBLISHED 8-Jun-2000 -> (none); PUBLISHER Altium Limited -> (none)
- U1: COMPONENTLINK1DESCRIPTION Manufacturer URL -> (none); COMPONENTLINK1URL http://www.microchip.com -> (none); COMPONENTLINK2DESCRIPTION Datasheet -> (none); COMPONENTLINK2URL http://ww1.microchip.com/downloads/en/DeviceDoc/70657F.pdf -> (none); COMPONENTLINK3DESCRIPTION Package Specification -> (none); COMPONENTLINK3URL http://www.microchip.com/stellent/groups/techpub_sg/documen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 -> (none); COMPONENTLINK4DESCRIPTION Product URL -> (none); COMPONENTLINK4URL http://www.microchip.com/dsPIC33EP256MC202 -> (none); DATASHEETVERSION Rev. F -> (none); MOUNTING TECHNOLOGY Through Hole -> (none); PACKAGEDESCRIPTION 28-Lead Plastic Dual In-Line, 34.86 x 6.79 mm Body, 2.54 mm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 -> (none); PACKAGEREFERENCE SPDIP-SP28 -> (none); PACKAGEVERSION C04-070B -> (none); PARTNUMBER DSPIC33EP256MC202-I/SP -> (none); SUPPLIER 1 Digi-Key -> (none); SUPPLIER 2 Farnell -> (none); SUPPLIER 3 Newark -> (none); SUPPLIER 4 Mouser -> (none); SUPPLIER PART NUMBER 1 DSPIC33EP256MC202-I/SP-ND -> (none); SUPPLIER PART NUMBER 2 2212194 -> (none); SUPPLIER PART NUMBER 3 66T8001 -> (none); SUPPLIER PART NUMBER 4 579-PC33256MC202ISP -> (none); now left out of the parts list
- U2: MFR_NAME Texas Instruments -> (none); REFDES RefDes -> (none); TYPE TYPE -> (none)
- U4: now left out of the parts list
